Commit message: Twister model

File: twister/ros/pt_description/urdf/pt.xacro (robot description, xacro)
@@ -4,151 +4,163 @@
   <!-- Constants for robot dimensions -->
   <xacro:property name="PI" value="3.1415926535897931"/>
-  <xacro:property name="mass" value="1" /> <!-- arbitrary value for mass -->
-  <xacro:property name="width" value="0.1" /> <!-- Square dimensions (widthxwidth) of beams -->
-  <xacro:property name="height1" value="2" /> <!-- Link 1 -->
-  <xacro:property name="height2" value="1" /> <!-- Link 2 -->
-  <xacro:property name="height3" value="1" /> <!-- Link 3 -->
-  <xacro:property name="camera_link" value="0.05" /> <!-- Size of square 'camera' box -->
-  <xacro:property name="axel_offset" value="0.05" /> <!-- Space btw top of beam and the each joint -->
   <!-- Import all Gazebo-customization elements, including Gazebo colors -->
   <xacro:include filename="$(find pt_description)/urdf/pt.gazebo" />
   <!-- Import Rviz colors -->
   <xacro:include filename="$(find pt_description)/urdf/materials.xacro" />
-  <!-- Used for fixing robot to Gazebo 'base_link' -->
-  <link name="world"/>
-  <joint name="fixed" type="fixed">
-    <parent link="world"/>
-    <child link="link1"/>
-  </joint>
-  <!-- Base Link -->
-  <link name="link1">
-    <collision>
-      <origin xyz="0 0 ${height1/2}" rpy="0 0 0"/>
-      <geometry>
-	<box size="${width} ${width} ${height1}"/>
-      </geometry>
-    </collision>
-    <visual>
-      <origin xyz="0 0 ${height1/2}" rpy="0 0 0"/>
-      <geometry>
-	<box size="${width} ${width} ${height1}"/>
+  <link name="base_link"/>
+  <joint name="chassis_joint" type="fixed">
+    <origin xyz="0.0 0.0 0.002"/>
+    <parent link="base_link"/>
+    <child link="chassis"/>
+  </joint>
+  <link name="chassis">
+    <visual>
+      <origin xyz="0 0 0" rpy="0 0 0"/>
+      <geometry>
+        <mesh filename="package://pt_description/meshes/twister_base.dae"/>
       </geometry>
       <material name="orange"/>
     </visual>
-    <inertial>
-      <origin xyz="0 0 ${height1/2}" rpy="0 0 0"/>
-      <mass value="${mass}"/>
-      <inertia
-	  ixx="${mass / 12.0 * (width*width + height1*height1)}" ixy="0.0" ixz="0.0"
-	  iyy="${mass / 12.0 * (height1*height1 + width*width)}" iyz="0.0"
-	  izz="${mass / 12.0 * (width*width + width*width)}"/>
-    </inertial>
-  </link>
-  <joint name="joint1" type="continuous">
-    <parent link="link1"/>
-    <child link="link2"/>
-    <origin xyz="0 ${width} ${height1 - axel_offset}" rpy="0 0 0"/>
-    <axis xyz="0 1 0"/>
-    <dynamics damping="0.7"/>
-  </joint>
-  <!-- Middle Link -->
-  <link name="link2">
-    <collision>
-      <origin xyz="0 0 ${height2/2 - axel_offset}" rpy="0 0 0"/>
-      <geometry>
-	<box size="${width} ${width} ${height2}"/>
-      </geometry>
-    </collision>
-    <visual>
-      <origin xyz="0 0 ${height2/2 - axel_offset}" rpy="0 0 0"/>
-      <geometry>
-	<box size="${width} ${width} ${height2}"/>
+    <collision>
+      <origin xyz="0.5 -0.015 0.062" rpy="0 0 0"/>
+      <geometry>
+        <box size="0.08 0.121 0.181"/>
+      </geometry>
+    </collision>
+    <inertial>
+      <origin xyz="0 -0.014693 0.06776" rpy="0 0 0"/>
+      <mass value="0.626"/>
+      <inertia ixx="6.154e-4" ixy="0.0" ixz="0.0"
+               iyy="4.298e-4" iyz="0.0"
+               izz="4.298e-4"/>
+    </inertial>
+  </link>
+  <joint name="right_wheel_hinge" type="continuous">
+    <parent link="chassis"/>
+    <child link="right_wheel_rim"/>
+    <origin xyz="0.0414 0 0.03255" rpy="0 0 0"/>
+    <axis xyz="1 0 0"/>
+    <dynamics damping="0.7" friction="0.0"/>
+  </joint>
+  <link name="right_wheel_rim">
+    <collision>
+      <origin xyz="0.017 0 0" rpy="0 1.5707 0"/>
+      <geometry>
+        <cylinder length="0.026" radius="0.032255"/>
+      </geometry>
+    </collision>
+    <visual>
+      <origin xyz="0 0 0" rpy="0 0 0"/>
+      <geometry>
+        <mesh filename="package://pt_description/meshes/twister_rim.dae"/>
+      </geometry>
+      <material name="yellow"/>
+    </visual>
+    <inertial>
+      <origin xyz="0.0179 0 0" rpy="0 0 0"/>
+      <mass value="0.010"/>
+      <inertia ixx="4.210e-8" ixy="0.0" ixz="0.0"
+               iyy="2.434e-8" iyz="0.0"
+               izz="2.434e-8"/>
+    </inertial>
+  </link>
+  <joint name="right_wheel_tire_mount" type="fixed">
+    <parent link="right_wheel_rim"/>
+    <child link="right_wheel_tire"/>
+  </joint>
+  <link name="right_wheel_tire">
+    <collision>
+      <origin xyz="0.017 0 0" rpy="0 1.5707 0"/>
+      <geometry>
+        <cylinder length="0.026" radius="0.032255"/>
+      </geometry>
+    </collision>
+    <visual>
+      <origin xyz="0 0 0" rpy="0 0 0"/>
+      <geometry>
+        <mesh filename="package://pt_description/meshes/twister_tire.dae"/>
       </geometry>
       <material name="black"/>
     </visual>
     <inertial>
-      <origin xyz="0 0 ${height2/2 - axel_offset}" rpy="0 0 0"/>
-      <mass value="${mass}"/>
-      <inertia
-	  ixx="${mass / 12.0 * (width*width + height2*height2)}" ixy="0.0" ixz="0.0"
-	  iyy="${mass / 12.0 * (height2*height2 + width*width)}" iyz="0.0"
-	  izz="${mass / 12.0 * (width*width + width*width)}"/>
-    </inertial>
-  </link>
-  <joint name="joint2" type="continuous">
-    <parent link="link2"/>
-    <child link="link3"/>
-    <origin xyz="0 ${width} ${height2 - axel_offset*2}" rpy="0 0 0"/>
-    <axis xyz="0 1 0"/>
-    <dynamics damping="0.7"/>
-  </joint>
-  <!-- Top Link -->
-  <link name="link3">
-    <collision>
-      <origin xyz="0 0 ${height3/2 - axel_offset}" rpy="0 0 0"/>
-      <geometry>
-	<box size="${width} ${width} ${height3}"/>
-      </geometry>
-    </collision>
-    <visual>
-      <origin xyz="0 0 ${height3/2 - axel_offset}" rpy="0 0 0"/>
-      <geometry>
-	<box size="${width} ${width} ${height3}"/>
-      </geometry>
-      <material name="orange"/>
-    </visual>
-    <inertial>
-      <origin xyz="0 0 ${height3/2 - axel_offset}" rpy="0 0 0"/>
-      <mass value="${mass}"/>
-      <inertia
-	  ixx="${mass / 12.0 * (width*width + height3*height3)}" ixy="0.0" ixz="0.0"
-	  iyy="${mass / 12.0 * (height3*height3 + width*width)}" iyz="0.0"
-	  izz="${mass / 12.0 * (width*width + width*width)}"/>
-    </inertial>
-  </link>
-  <joint name="hokuyo_joint" type="fixed">
-    <axis xyz="0 1 0" />
-    <origin xyz="0 0 ${height3 - axel_offset/2}" rpy="0 0 0"/>
-    <parent link="link3"/>
-    <child link="hokuyo_link"/>
-  </joint>
-  <!-- Hokuyo Laser -->
-  <link name="hokuyo_link">
-    <collision>
-      <origin xyz="0 0 0" rpy="0 0 0"/>
-      <geometry>
-	<box size="0.1 0.1 0.1"/>
-      </geometry>
-    </collision>
-    <visual>
-      <origin xyz="0 0 0" rpy="0 0 0"/>
-      <geometry>
-        <mesh filename="package://pt_description/meshes/hokuyo.dae"/>
-      </geometry>
-    </visual>
-    <inertial>
-      <mass value="1e-5" />
-      <origin xyz="0 0 0" rpy="0 0 0"/>
-      <inertia ixx="1e-6" ixy="0" ixz="0" iyy="1e-6" iyz="0" izz="1e-6" />
+      <origin xyz="0.0179 0 0" rpy="0 0 0"/>
+      <mass value="0.057"/>
+      <inertia ixx="4.210e-5" ixy="0.0" ixz="0.0"
+               iyy="2.434e-5" iyz="0.0"
+               izz="2.434e-5"/>
+    </inertial>
+  </link>
+  <joint name="left_wheel_hinge" type="continuous">
+    <parent link="chassis"/>
+    <child link="left_wheel_rim"/>
+    <origin xyz="-0.0414 0 0.03255" rpy="0 0 3.14159"/>
+    <axis xyz="1 0 0"/>
+    <dynamics damping="0.7" friction="0"/>
+  </joint>
+  <link name="left_wheel_rim">
+    <collision>
+      <origin xyz="0.017 0 0" rpy="0 1.5707 0"/>
+      <geometry>
+        <cylinder length="0.026" radius="0.032255"/>
+      </geometry>
+    </collision>
+    <visual>
+      <origin xyz="0 0 0" rpy="0 0 0"/>
+      <geometry>
+        <mesh filename="package://pt_description/meshes/twister_rim.dae"/>
+      </geometry>
+      <material name="yellow"/>
+    </visual>
+    <inertial>
+      <origin xyz="0.0179 0 0" rpy="0 0 0"/>
+      <mass value="0.010"/>
+      <inertia ixx="4.210e-8" ixy="0.0" ixz="0.0"
+               iyy="2.434e-8" iyz="0.0"
+               izz="2.434e-8"/>
+    </inertial>
+  </link>
+  <joint name="left_wheel_tire_mount" type="fixed">
+    <parent link="left_wheel_rim"/>
+    <child link="left_wheel_tire"/>
+  </joint>
+  <link name="left_wheel_tire">
+    <collision>
+      <origin xyz="0.017 0 0" rpy="0 1.5707 0"/>
+      <geometry>
+        <cylinder length="0.026" radius="0.032255"/>
+      </geometry>
+    </collision>
+    <visual>
+      <origin xyz="0 0 0" rpy="0 0 0"/>
+      <geometry>
+        <mesh filename="package://pt_description/meshes/twister_tire.dae"/>
+      </geometry>
+      <material name="black"/>
+    </visual>
+    <inertial>
+      <origin xyz="0.0179 0 0" rpy="0 0 0"/>
+      <mass value="0.057"/>
+      <inertia ixx="4.210e-5" ixy="0.0" ixz="0.0"
+               iyy="2.434e-5" iyz="0.0"
+               izz="2.434e-5"/>
     </inertial>
   </link>
   <joint name="camera_joint" type="fixed">
     <axis xyz="0 1 0" />
-    <origin xyz="${camera_link} 0 ${height3 - axel_offset*2}" rpy="0 0 0"/>
-    <parent link="link3"/>
+    <origin xyz="0 0.045 0.090" rpy="0 0 0"/>
+    <parent link="chassis"/>
     <child link="camera_link"/>
   </joint>
-  <!-- Camera -->
   <link name="camera_link">
     <collision>
       <origin xyz="0 0 0" rpy="0 0 0"/>
       <geometry>
-	<box size="${camera_link} ${camera_link} ${camera_link}"/>
-      </geometry>
-    </collision>
-    <visual>
-      <origin xyz="0 0 0" rpy="0 0 0"/>
-      <geometry>
-	<box size="${camera_link} ${camera_link} ${camera_link}"/>
+        <box size="0.005 0.005 0.005"/>
+      </geometry>
+    </collision>
+    <visual>
+      <origin xyz="0 0 0" rpy="0 0 0"/>
+      <geometry>
+        <box size="0.005 0.005 0.005"/>
       </geometry>
       <material name="red"/>
@@ -157,5 +169,7 @@
       <mass value="1e-5" />
       <origin xyz="0 0 0" rpy="0 0 0"/>
-      <inertia ixx="1e-6" ixy="0" ixz="0" iyy="1e-6" iyz="0" izz="1e-6" />
+      <inertia ixx="1e-8" ixy="0" ixz="0"
+               iyy="1e-8" iyz="0"
+               izz="1e-8" />
     </inertial>
   </link>
@@ -171,22 +185,20 @@
   <link name="camera_link_optical">
   </link>
-  <transmission name="tran1">
+  <transmission name="right_wheel_transmission" type="SimpleTransmission">
     <type>transmission_interface/SimpleTransmission</type>
-    <joint name="joint1">
+    <joint name="right_wheel_hinge">
       <hardwareInterface>hardware_interface/EffortJointInterface</hardwareInterface>
     </joint>
-    <actuator name="motor1">
-      <hardwareInterface>hardware_interface/EffortJointInterface</hardwareInterface>
-      <mechanicalReduction>1</mechanicalReduction>
+    <actuator name="right_wheel_motor">
+      <mechanicalReduction>48</mechanicalReduction>
     </actuator>
   </transmission>
-  <transmission name="tran2">
+  <transmission name="left_wheel_transmission" type="SimpleTransmission">
     <type>transmission_interface/SimpleTransmission</type>
-    <joint name="joint2">
+    <joint name="left_wheel_hinge">
       <hardwareInterface>hardware_interface/EffortJointInterface</hardwareInterface>
     </joint>
-    <actuator name="motor2">
-      <hardwareInterface>hardware_interface/EffortJointInterface</hardwareInterface>
-      <mechanicalReduction>1</mechanicalReduction>
+    <actuator name="left_wheel_motor">
+      <mechanicalReduction>48</mechanicalReduction>
     </actuator>
   </transmission>

Commit message: ODE Stability

File: twister/ros/pt_description/urdf/pt.xacro (robot description, xacro)
@@ -4,15 +4,22 @@
   <!-- Constants for robot dimensions -->
   <xacro:property name="PI" value="3.1415926535897931"/>
+  <xacro:property name="mass" value="0.06" /> <!-- arbitrary value for mass -->
+  <xacro:property name="width" value="0.015" /> <!-- Square dimensions (widthxwidth) of beams -->
+  <xacro:property name="height1" value="0.3" /> <!-- Link 1 -->
+  <xacro:property name="height2" value="0.05" /> <!-- Link 2 -->
+  <xacro:property name="height3" value="0.05" /> <!-- Link 3 -->
+  <xacro:property name="camera_link" value="0.0125" /> <!-- Size of square 'camera' box -->
+  <xacro:property name="axel_offset" value="0.0125" /> <!-- Space btw top of beam and the each joint -->
   <!-- Import all Gazebo-customization elements, including Gazebo colors -->
   <xacro:include filename="$(find pt_description)/urdf/pt.gazebo" />
   <!-- Import Rviz colors -->
   <xacro:include filename="$(find pt_description)/urdf/materials.xacro" />
-  <link name="base_link"/>
-  <joint name="chassis_joint" type="fixed">
-    <origin xyz="0.0 0.0 0.002"/>
-    <parent link="base_link"/>
-    <child link="chassis"/>
-  </joint>
   <link name="chassis">
+    <collision>
+      <origin xyz="0.0 -0.015 0.0615" rpy="0 0 0"/>
+      <geometry>
+        <box size="0.08 0.121 0.085"/>
+      </geometry>
+    </collision>
     <visual>
       <origin xyz="0 0 0" rpy="0 0 0"/>
@@ -22,10 +29,4 @@
       <material name="orange"/>
     </visual>
-    <collision>
-      <origin xyz="0.5 -0.015 0.062" rpy="0 0 0"/>
-      <geometry>
-        <box size="0.08 0.121 0.181"/>
-      </geometry>
-    </collision>
     <inertial>
       <origin xyz="0 -0.014693 0.06776" rpy="0 0 0"/>
@@ -36,4 +37,62 @@
     </inertial>
   </link>
+  <joint name="back_wheel_holder_hinge" type="continuous">
+    <parent link="chassis"/>
+    <child link="back_wheel_holder"/>
+    <origin xyz="0.0 -0.0687 0.0183" rpy="0 0 0"/>
+    <axis xyz="0 0 1"/>
+    <dynamics damping="0.01" friction="0.01"/>
+  </joint>
+  <link name="back_wheel_holder">
+    <collision>
+      <origin xyz="0 -0.009 -0.0065" rpy="0 0 0"/>
+      <geometry>
+        <box size="0.012 0.024 0.013"/>
+      </geometry>
+    </collision>
+    <visual>
+      <origin xyz="0 0 0" rpy="0 0 0"/>
+      <geometry>
+        <mesh filename="package://pt_description/meshes/twister_back_wheel_holder.dae"/>
+      </geometry>
+      <material name="yellow"/>
+    </visual>
+    <inertial>
+      <origin xyz="0 -0.008 -0.0046" rpy="0 0 0"/>
+      <mass value="0.001"/>
+      <inertia ixx="7.198e-8" ixy="0.0" ixz="0.0"
+               iyy="3.400e-8" iyz="0.0"
+               izz="8.483e-8"/>
+    </inertial>
+  </link>
+  <joint name="back_wheel_hinge" type="continuous">
+    <parent link="back_wheel_holder"/>
+    <child link="back_wheel"/>
+    <origin xyz="0.0 -0.016 -0.008" rpy="0 0 0"/>
+    <axis xyz="1 0 0"/>
+    <dynamics damping="0.01" friction="0.001"/>
+  </joint>
+  <link name="back_wheel">
+    <collision>
+      <origin xyz="0 0 0" rpy="0 1.5707 0"/>
+      <geometry>
+        <cylinder length="0.007" radius="0.0075"/>
+      </geometry>
+    </collision>
+    <visual>
+      <origin xyz="0 0 0" rpy="0 0 0"/>
+      <geometry>
+        <mesh filename="package://pt_description/meshes/twister_back_wheel.dae"/>
+      </geometry>
+      <material name="yellow"/>
+    </visual>
+    <inertial>
+      <origin xyz="0 0 0" rpy="0 0 0"/>
+      <mass value="0.001"/>
+      <inertia ixx="2.427e-8" ixy="0.0" ixz="0.0"
+               iyy="1.393e-8" iyz="0.0"
+               izz="1.393e-8"/>
+    </inertial>
+  </link>
   <joint name="right_wheel_hinge" type="continuous">
     <parent link="chassis"/>
@@ -41,11 +100,11 @@
     <origin xyz="0.0414 0 0.03255" rpy="0 0 0"/>
     <axis xyz="1 0 0"/>
-    <dynamics damping="0.7" friction="0.0"/>
+    <dynamics damping="0.001"/>
   </joint>
   <link name="right_wheel_rim">
     <collision>
-      <origin xyz="0.017 0 0" rpy="0 1.5707 0"/>
-      <geometry>
-        <cylinder length="0.026" radius="0.032255"/>
+      <origin xyz="0.016 0 0" rpy="0 1.5707 0"/>
+      <geometry>
+        <cylinder length="0.027" radius="0.032255"/>
       </geometry>
     </collision>
@@ -71,7 +130,7 @@
   <link name="right_wheel_tire">
     <collision>
-      <origin xyz="0.017 0 0" rpy="0 1.5707 0"/>
-      <geometry>
-        <cylinder length="0.026" radius="0.032255"/>
+      <origin xyz="0.016 0 0" rpy="0 1.5707 0"/>
+      <geometry>
+        <cylinder length="0.027" radius="0.032255"/>
       </geometry>
     </collision>
@@ -84,6 +143,6 @@
     </visual>
     <inertial>
-      <origin xyz="0.0179 0 0" rpy="0 0 0"/>
-      <mass value="0.057"/>
+      <origin xyz="0.016 0 0" rpy="0 0 0"/>
+      <mass value="0.047"/>
       <inertia ixx="4.210e-5" ixy="0.0" ixz="0.0"
                iyy="2.434e-5" iyz="0.0"
@@ -91,4 +150,34 @@
     </inertial>
   </link>
+  <joint name="joint2" type="fixed">
+    <parent link="right_wheel_rim"/>
+    <child link="right_wheel_tire2"/>
+    <origin xyz="0.03 0 0.05" rpy="0 0 0"/>
+    <axis xyz="0 1 0"/>
+    <dynamics damping="0.001"/>
+  </joint>
+  <link name="right_wheel_tire2">
+    <collision>
+      <origin xyz="0 0 ${height3/2 - axel_offset}" rpy="0 0 0"/>
+      <geometry>
+        <box size="${width} ${width} ${height3}"/>
+      </geometry>
+    </collision>
+    <visual>
+      <origin xyz="0 0 ${height3/2 - axel_offset}" rpy="0 0 0"/>
+      <geometry>
+        <box size="${width} ${width} ${height3}"/>
+      </geometry>
+      <material name="yellow"/>
+    </visual>
+    <inertial>
+      <origin xyz="0 0 ${height3/2 - axel_offset}" rpy="0 0 0"/>
+      <mass value="${mass}"/>
+      <inertia
+    ixx="${mass / 12.0 * (width*width + height3*height3)}" ixy="0.0" ixz="0.0"
+    iyy="${mass / 12.0 * (height3*height3 + width*width)}" iyz="0.0"
+    izz="${mass / 12.0 * (width*width + width*width)}"/>
+    </inertial>
+  </link>
   <joint name="left_wheel_hinge" type="continuous">
     <parent link="chassis"/>
@@ -96,13 +185,7 @@
     <origin xyz="-0.0414 0 0.03255" rpy="0 0 3.14159"/>
     <axis xyz="1 0 0"/>
-    <dynamics damping="0.7" friction="0"/>
+    <dynamics damping="0.001"/>
   </joint>
   <link name="left_wheel_rim">
-    <collision>
-      <origin xyz="0.017 0 0" rpy="0 1.5707 0"/>
-      <geometry>
-        <cylinder length="0.026" radius="0.032255"/>
-      </geometry>
-    </collision>
     <visual>
       <origin xyz="0 0 0" rpy="0 0 0"/>
@@ -126,7 +209,7 @@
   <link name="left_wheel_tire">
     <collision>
-      <origin xyz="0.017 0 0" rpy="0 1.5707 0"/>
-      <geometry>
-        <cylinder length="0.026" radius="0.032255"/>
+      <origin xyz="0.016 0 0" rpy="0 1.5707 0"/>
+      <geometry>
+        <cylinder length="0.027" radius="0.032255"/>
       </geometry>
     </collision>
@@ -139,6 +222,6 @@
     </visual>
     <inertial>
-      <origin xyz="0.0179 0 0" rpy="0 0 0"/>
-      <mass value="0.057"/>
+      <origin xyz="0.016 0 0" rpy="0 0 0"/>
+      <mass value="0.047"/>
       <inertia ixx="4.210e-5" ixy="0.0" ixz="0.0"
                iyy="2.434e-5" iyz="0.0"
@@ -148,5 +231,5 @@
   <joint name="camera_joint" type="fixed">
     <axis xyz="0 1 0" />
-    <origin xyz="0 0.045 0.090" rpy="0 0 0"/>
+    <origin xyz="0 0.05 0.090" rpy="0 0 0"/>
     <parent link="chassis"/>
     <child link="camera_link"/>
@@ -174,10 +257,6 @@
     </inertial>
   </link>
-  <!-- generate an optical frame http://www.ros.org/reps/rep-0103.html#suffix-frames
-      so that ros and opencv can operate on the camera frame correctly -->
   <joint name="camera_optical_joint" type="fixed">
-    <!-- these values have to be these values otherwise the gazebo camera image
-        won't be aligned properly with the frame it is supposedly originating from -->
-    <origin xyz="0 0 0" rpy="${-pi/2} 0 ${-pi/2}"/>
+    <origin xyz="0 0 0" rpy="${-PI/2} 0 ${-PI/2}"/>
     <parent link="camera_link"/>
     <child link="camera_link_optical"/>
@@ -191,5 +270,5 @@
     </joint>
     <actuator name="right_wheel_motor">
-      <mechanicalReduction>48</mechanicalReduction>
+      <mechanicalReduction>1</mechanicalReduction>
     </actuator>
   </transmission>
@@ -200,5 +279,5 @@
     </joint>
     <actuator name="left_wheel_motor">
-      <mechanicalReduction>48</mechanicalReduction>
+      <mechanicalReduction>1</mechanicalReduction>
     </actuator>
   </transmission>
