Commit message: Correct textures

File: twister/ros/pt_description/urdf/pt.xacro (robot description, xacro)
@@ -15,4 +15,11 @@
   <!-- Import Rviz colors -->
   <xacro:include filename="$(find pt_description)/urdf/materials.xacro" />
+  <link name="puffin">
+  </link>
+  <joint name="chassis_fix" type="fixed">
+    <parent link="puffin"/>
+    <child link="chassis"/>
+    <origin xyz="0.45 0.30 0" rpy="0 0 0"/>
+  </joint>
   <link name="chassis">
     <collision>
@@ -25,5 +32,5 @@
       <origin xyz="0 0 0" rpy="0 0 0"/>
       <geometry>
-        <mesh filename="package://pt_description/meshes/twister_base.dae"/>
+        <mesh filename="package://pt_description/meshes/twister_base.stl"/>
       </geometry>
       <material name="orange"/>
@@ -52,5 +59,5 @@
       <origin xyz="0 0 0" rpy="0 0 0"/>
       <geometry>
-        <mesh filename="package://pt_description/meshes/twister_camera_holder.dae"/>
+        <mesh filename="package://pt_description/meshes/twister_camera_holder.stl"/>
       </geometry>
       <material name="orange"/>
@@ -79,5 +86,5 @@
       <origin xyz="0 0 0" rpy="0 0 0"/>
       <geometry>
-        <mesh filename="package://pt_description/meshes/twister_motor.dae"/>
+        <mesh filename="package://pt_description/meshes/twister_motor.stl"/>
       </geometry>
       <material name="orange"/>
@@ -106,5 +113,5 @@
       <origin xyz="0 0 0" rpy="0 0 0"/>
       <geometry>
-        <mesh filename="package://pt_description/meshes/twister_motor.dae"/>
+        <mesh filename="package://pt_description/meshes/twister_motor.stl"/>
       </geometry>
       <material name="orange"/>
@@ -133,5 +140,5 @@
       <origin xyz="0 0 0" rpy="0 0 0"/>
       <geometry>
-        <mesh filename="package://pt_description/meshes/twister_battery_holder.dae"/>
+        <mesh filename="package://pt_description/meshes/twister_battery_holder.stl"/>
       </geometry>
       <material name="orange"/>
@@ -160,5 +167,5 @@
       <origin xyz="0 0 0" rpy="0 0 0"/>
       <geometry>
-        <mesh filename="package://pt_description/meshes/twister_battery_holder.dae"/>
+        <mesh filename="package://pt_description/meshes/twister_battery_holder.stl"/>
       </geometry>
       <material name="orange"/>
@@ -189,5 +196,5 @@
       <origin xyz="0 0 0" rpy="0 0 0"/>
       <geometry>
-        <mesh filename="package://pt_description/meshes/twister_back_wheel_holder.dae"/>
+        <mesh filename="package://pt_description/meshes/twister_back_wheel_holder.stl"/>
       </geometry>
       <material name="yellow"/>
@@ -218,5 +225,5 @@
       <origin xyz="0 0 0" rpy="0 0 0"/>
       <geometry>
-        <mesh filename="package://pt_description/meshes/twister_back_wheel.dae"/>
+        <mesh filename="package://pt_description/meshes/twister_back_wheel.stl"/>
       </geometry>
       <material name="yellow"/>
@@ -234,5 +241,5 @@
     <child link="right_wheel_rim"/>
     <origin xyz="0.0414 0 0.03255" rpy="0 0 0"/>
-    <axis xyz="1 0 0"/>
+    <axis xyz="-1 0 0"/>
     <dynamics damping="0.01" friction="0.001"/>
   </joint>
@@ -247,5 +254,5 @@
       <origin xyz="0 0 0" rpy="0 0 0"/>
       <geometry>
-        <mesh filename="package://pt_description/meshes/twister_rim.dae"/>
+        <mesh filename="package://pt_description/meshes/twister_rim.stl"/>
       </geometry>
       <material name="yellow"/>
@@ -273,5 +280,5 @@
       <origin xyz="0 0 0" rpy="0 0 0"/>
       <geometry>
-        <mesh filename="package://pt_description/meshes/twister_tire.dae"/>
+        <mesh filename="package://pt_description/meshes/twister_tire.stl"/>
       </geometry>
       <material name="black"/>
@@ -296,5 +303,5 @@
       <origin xyz="0 0 0" rpy="0 0 0"/>
       <geometry>
-        <mesh filename="package://pt_description/meshes/twister_rim.dae"/>
+        <mesh filename="package://pt_description/meshes/twister_rim.stl"/>
       </geometry>
       <material name="yellow"/>
@@ -322,5 +329,5 @@
       <origin xyz="0 0 0" rpy="0 0 0"/>
       <geometry>
-        <mesh filename="package://pt_description/meshes/twister_tire.dae"/>
+        <mesh filename="package://pt_description/meshes/twister_tire.stl"/>
       </geometry>
       <material name="black"/>
